Commit message: [feta]:添加gazebo仿真支持

File: src/fishbot_description/urdf/fishbot_base.urdf (robot description, URDF)
Before this commit: robot fishbot, 3 links, 2 joints
Links:
- added link base_footprint; visual box size=0.001 0.001 0.001
- added link caster_link; visual sphere radius=0.016
- added link left_wheel_link; visual cylinder length=0.04 radius=0.032
- added link right_wheel_link; visual cylinder length=0.04 radius=0.032
Joints:
- added joint caster_joint: type fixed, parent base_link, child caster_link, origin xyz=0.06 0.0 -0.076, axis 0 1 0
- added joint left_wheel_joint: type continuous, parent base_link, child left_wheel_link, origin xyz=-0.02 -0.10 -0.06, axis 0 1 0
- added joint right_wheel_joint: type continuous, parent base_link, child right_wheel_link, origin xyz=-0.02 0.10 -0.06, axis 0 1 0

Commit message: [fix]:修复一些错误

File: src/fishbot_description/urdf/fishbot_base.urdf (robot description, URDF)
Before this commit: robot fishbot, 7 links, 5 joints
Links:
- removed link base_footprint
Joints:
- joint left_wheel_joint: origin xyz=-0.02 -0.10 -0.06 -> xyz=-0.02 0.10 -0.06
- joint right_wheel_joint: origin xyz=-0.02 0.10 -0.06 -> xyz=-0.02 -0.10 -0.06
