Commit message: [feta]:add navigation2

File: src/fishbot_description/urdf/fishbot_gazebo.urdf (robot description, URDF)
Before this commit: robot fishbot, 6 links, 5 joints
Links:
- added link base_footprint
Joints:
- added joint base_joint: type fixed, parent base_footprint, child base_link, origin xyz=0.0 0.0 0.076 rpy=0 0 0
- joint left_wheel_joint: axis 0 1 0 -> 0.0 1 0

Commit message: [feta]:基本调试完成fishbot建图与导航

File: src/fishbot_description/urdf/fishbot_gazebo.urdf (robot description, URDF)
Before this commit: robot fishbot, 7 links, 6 joints
Joints:
- joint left_wheel_joint: axis 0.0 1 0 -> 0 1 0; origin xyz=-0.02 -0.10 -0.06 -> xyz=-0.02 0.10 -0.06
- joint right_wheel_joint: origin xyz=-0.02 0.10 -0.06 -> xyz=-0.02 -0.10 -0.06
